File: Interfacebox module board.kicad_pcb (KiCad board)
At the start: 2 copper layers, 319.7 x 109.8 mm, 70 parts, among them J1 Malfboard bottom, J2 Malfboard top, J3 Driverboard_malf-board, J4 Driverboard_TR-switch

Commit message: Added: connectors to distribute 16ch to 2 boards
Parts:
- added J5: 1-8, Connector_IDC:IDC-Header_2x04_P2.54mm_Vertical, F.Cu at (292.0, 85.8)
- added J6: 9-16, Connector_IDC:IDC-Header_2x04_P2.54mm_Vertical, F.Cu at (292.0, 99.6)
- added L1: choke, Inductor_SMD:L_1812_4532Metric, F.Cu at (261.6, 80.6)
- added L10: choke, Inductor_SMD:L_1812_4532Metric, F.Cu at (267.6, 92.6)
- added L11: choke, Inductor_SMD:L_1812_4532Metric, F.Cu at (273.6, 95.0)
- added L12: choke, Inductor_SMD:L_1812_4532Metric, F.Cu at (279.6, 97.4)
- added L13: choke, Inductor_SMD:L_1812_4532Metric, F.Cu at (261.6, 95.0)
- added L14: choke, Inductor_SMD:L_1812_4532Metric, F.Cu at (267.6, 97.4)
- added L15: choke, Inductor_SMD:L_1812_4532Metric, F.Cu at (273.6, 99.8)
- added L16: choke, Inductor_SMD:L_1812_4532Metric, F.Cu at (279.6, 102.2)
- added L2: choke, Inductor_SMD:L_1812_4532Metric, F.Cu at (267.6, 83.0)
- added L3: choke, Inductor_SMD:L_1812_4532Metric, F.Cu at (273.6, 85.4)
- added L4: choke, Inductor_SMD:L_1812_4532Metric, F.Cu at (279.6, 87.8)
- added L5: choke, Inductor_SMD:L_1812_4532Metric, F.Cu at (261.6, 85.4)
- added L6: choke, Inductor_SMD:L_1812_4532Metric, F.Cu at (267.6, 87.8)
- added L7: choke, Inductor_SMD:L_1812_4532Metric, F.Cu at (273.6, 90.2)
- added L8: choke, Inductor_SMD:L_1812_4532Metric, F.Cu at (279.6, 92.6)
- added L9: choke, Inductor_SMD:L_1812_4532Metric, F.Cu at (261.6, 90.2)
- moved G1 34.9 mm to (324.0, 92.6)
Routing:
- net Net-(Ch1-Pad1): track 117.7 -> 255.4 mm
- net Net-(Ch2-Pad1): track 111.5 -> 247.3 mm
- net Net-(Ch3-Pad1): track 30.3 -> 163.7 mm, vias 0 -> 2
- net Net-(Ch4-Pad1): track 104.0 -> 236.0 mm, vias 1 -> 3
- net Net-(Ch5-Pad1): track 48.9 -> 155.4 mm
- net Net-(Ch6-Pad1): track 105.5 -> 209.7 mm
- net Net-(Ch7-Pad1): track 63.1 -> 165.6 mm, vias 1 -> 3
- net Net-(Ch8-Pad1): track 121.5 -> 222.9 mm, vias 1 -> 3
- net Net-(Ch9-Pad1): track 18.7 -> 93.7 mm
- net Net-(Ch10-Pad1): track 86.0 -> 158.6 mm
- net Net-(Ch11-Pad1): track 19.1 -> 90.5 mm, vias 1 -> 3
- net Net-(Ch12-Pad1): track 110.9 -> 180.7 mm, vias 0 -> 2
- net Net-(Ch13-Pad1): track 19.6 -> 63.0 mm
- net Net-(Ch14-Pad1): track 134.6 -> 176.0 mm
- net Net-(Ch15-Pad1): track 18.4 -> 58.5 mm
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Other:
- board text added: "02/2020 v0.2"
- board text added: "Connect J6 on master to J5 on slave board to make 16ch with 1 driver/malfunction board"
- board text added: "Preamp board ook modulair? Handig bij 'recycling' van box/preampboard gaten in pcb voor connectors geen top ground waar module komt (tegen spikes)"
- board text added: "ch1-8"
- board text added: "ch9-16"
- board text removed: "02/2020 v0.1"
