File: Interfacebox module board.kicad_pcb (KiCad board)
At the start: 2 copper layers, 319.7 x 109.8 mm, 88 parts, among them J1 Malfboard bottom, J2 Malfboard top, J3 Driverboard_malf-board, J4 Driverboard_TR-switch, J5 1-8, J6 9-16

Commit message: Changed: comments; README. Added: 3D render
Other:
- board text added: "35.5cm current box (+4cm on side for cable) 1-2cm less wide would fir better 35.5 - 1 = 34.5 (housing = 1cm) 34.5 - 2 = 32.5cm pcb"
- board text removed: "35.5cm is box nu aan buitenkant (+4cm voor zijkant kabel uitsteeksel) Hans: 1-2cm minder breed is fijn 35.5 - 1 = 34.5 (door behuizing) 34.5 - 2 = 32.5cm pcb?"
- board text removed: "Preamp board ook modulair? Handig bij 'recycling' van box/preampboard gaten in pcb voor connectors geen top ground waar module komt (tegen spikes)"
Changed lines of the file:
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@@
   (general
     (thickness 1.6)
-    (drawings 129)
+    (drawings 106)
     (tracks 535)
     (zones 0)
@@
   (gr_line (start 362.979999 185.8) (end 45.870001 185.800001) (layer Edge.Cuts) (width 0.05))
   (dimension 9.75 (width 0.12) (layer Cmts.User)
-    (gr_text "9.750 mm" (at 355.575 197.07) (layer Cmts.User)
-      (effects (font (size 1 1) (thickness 0.15)))
-    )
-    (feature1 (pts (xy 350.7 191.5) (xy 350.7 196.386421)))
-    (feature2 (pts (xy 360.45 191.5) (xy 360.45 196.386421)))
-    (crossbar (pts (xy 360.45 195.8) (xy 350.7 195.8)))
-    (arrow1a (pts (xy 350.7 195.8) (xy 351.826504 195.213579)))
-    (arrow1b (pts (xy 350.7 195.8) (xy 351.826504 196.386421)))
-    (arrow2a (pts (xy 360.45 195.8) (xy 359.323496 195.213579)))
-    (arrow2b (pts (xy 360.45 195.8) (xy 359.323496 196.386421)))
-  )
-  (dimension 9.75 (width 0.12) (layer Cmts.User)
     (gr_text "9.750 mm" (at 53.325 197.07) (layer Cmts.User)
       (effects (font (size 1 1) (thickness 0.15)))
     )
-    (feature1 (pts (xy 48.45 191.5) (xy 48.45 196.386421)))
-    (feature2 (pts (xy 58.2 191.5) (xy 58.2 196.386421)))
+    (feature1 (pts (xy 48.45 190) (xy 48.45 196.386421)))
+    (feature2 (pts (xy 58.2 190) (xy 58.2 196.386421)))
     (crossbar (pts (xy 58.2 195.8) (xy 48.45 195.8)))
     (arrow1a (pts (xy 48.45 195.8) (xy 49.576504 195.213579)))
@@
   )
   (dimension 39 (width 0.12) (layer Cmts.User)
-    (gr_text "8ch: 39.000 mm" (at 312.15 202.019999) (layer Cmts.User)
-      (effects (font (size 1 1) (thickness 0.15)))
-    )
-    (feature1 (pts (xy 331.65 193.25) (xy 331.65 201.33642)))
-    (feature2 (pts (xy 292.65 193.25) (xy 292.65 201.33642)))
-    (crossbar (pts (xy 292.65 200.749999) (xy 331.65 200.749999)))
-    (arrow1a (pts (xy 331.65 200.749999) (xy 330.523496 201.33642)))
-    (arrow1b (pts (xy 331.65 200.749999) (xy 330.523496 200.163578)))
-    (arrow2a (pts (xy 292.65 200.749999) (xy 293.776504 201.33642)))
-    (arrow2b (pts (xy 292.65 200.749999) (xy 293.776504 200.163578)))
-  )
-  (dimension 39 (width 0.12) (layer Cmts.User)
-    (gr_text "8ch: 39.000 mm" (at 273.15 210.369999) (layer Cmts.User)
+    (gr_text "1.5354 in" (at 77.7 198.87) (layer Cmts.User)
       (effects (font (size 1 1) (thickness 0.15)))
     )
-    (feature1 (pts (xy 292.65 201.6) (xy 292.65 209.68642)))
-    (feature2 (pts (xy 253.65 201.6) (xy 253.65 209.68642)))
-    (crossbar (pts (xy 253.65 209.099999) (xy 292.65 209.099999)))
-    (arrow1a (pts (xy 292.65 209.099999) (xy 291.523496 209.68642)))
-    (arrow1b (pts (xy 292.65 209.099999) (xy 291.523496 208.513578)))
-    (arrow2a (pts (xy 253.65 209.099999) (xy 254.776504 209.68642)))
-    (arrow2b (pts (xy 253.65 209.099999) (xy 254.776504 208.513578)))
-  )
-  (dimension 39 (width 0.12) (layer Cmts.User)
-    (gr_text "8ch: 39.000 mm" (at 233.8 201.469999) (layer Cmts.User)
-      (effects (font (size 1 1) (thickness 0.15)))
-    )
-    (feature1 (pts (xy 253.3 192.7) (xy 253.3 200.78642)))
-    (feature2 (pts (xy 214.3 192.7) (xy 214.3 200.78642)))
-    (crossbar (pts (xy 214.3 200.199999) (xy 253.3 200.199999)))
-    (arrow1a (pts (xy 253.3 200.199999) (xy 252.173496 200.78642)))
-    (arrow1b (pts (xy 253.3 200.199999) (xy 252.173496 199.613578)))
-    (arrow2a (pts (xy 214.3 200.199999) (xy 215.426504 200.78642)))
-    (arrow2b (pts (xy 214.3 200.199999) (xy 215.426504 199.613578)))
-  )
-  (dimension 39 (width 0.12) (layer Cmts.User)
-    (gr_text "8ch: 39.000 mm" (at 195.3 210.169999) (layer Cmts.User)
-      (effects (font (size 1 1) (thickness 0.15)))
-    )
-    (feature1 (pts (xy 214.8 201.4) (xy 214.8 209.48642)))
-    (feature2 (pts (xy 175.8 201.4) (xy 175.8 209.48642)))
-    (crossbar (pts (xy 175.8 208.899999) (xy 214.8 208.899999)))
-    (arrow1a (pts (xy 214.8 208.899999) (xy 213.673496 209.48642)))
-    (arrow1b (pts (xy 214.8 208.899999) (xy 213.673496 208.313578)))
-    (arrow2a (pts (xy 175.8 208.899999) (xy 176.926504 209.48642)))
-    (arrow2b (pts (xy 175.8 208.899999) (xy 176.926504 208.313578)))
-  )
-  (dimension 39 (width 0.12) (layer Cmts.User)
-    (gr_text "8ch: 39.000 mm" (at 155.95 201.819999) (layer Cmts.User)
-      (effects (font (size 1 1) (thickness 0.15)))
-    )
-    (feature1 (pts (xy 175.45 193.05) (xy 175.45 201.13642)))
-    (feature2 (pts (xy 136.45 193.05) (xy 136.45 201.13642)))
-    (crossbar (pts (xy 136.45 200.549999) (xy 175.45 200.549999)))
-    (arrow1a (pts (xy 175.45 200.549999) (xy 174.323496 201.13642)))
-    (arrow1b (pts (xy 175.45 200.549999) (xy 174.323496 199.963578)))
-    (arrow2a (pts (xy 136.45 200.549999) (xy 137.576504 201.13642)))
-    (arrow2b (pts (xy 136.45 200.549999) (xy 137.576504 199.963578)))
-  )
-  (dimension 39 (width 0.12) (layer Cmts.User)
-    (gr_text "8ch: 39.000 mm" (at 116.9 208.219999) (layer Cmts.User)
-      (effects (font (size 1 1) (thickness 0.15)))
-    )
-    (feature1 (pts (xy 136.4 199.45) (xy 136.4 207.53642)))
-    (feature2 (pts (xy 97.4 199.45) (xy 97.4 207.53642)))
-    (crossbar (pts (xy 97.4 206.949999) (xy 136.4 206.949999)))
-    (arrow1a (pts (xy 136.4 206.949999) (xy 135.273496 207.53642)))
-    (arrow1b (pts (xy 136.4 206.949999) (xy 135.273496 206.363578)))
-    (arrow2a (pts (xy 97.4 206.949999) (xy 98.526504 207.53642)))
-    (arrow2b (pts (xy 97.4 206.949999) (xy 98.526504 206.363578)))
-  )
-  (gr_line (start 350.7 191.5) (end 350.7 190) (layer Cmts.User) (width 0.12))
-  (dimension 39 (width 0.12) (layer Cmts.User)
-    (gr_text "8ch: 39.000 mm" (at 77.7 198.769999) (layer Cmts.User)
-      (effects (font (size 1 1) (thickness 0.15)))
-    )
-    (feature1 (pts (xy 97.2 190) (xy 97.2 198.08642)))
-    (feature2 (pts (xy 58.2 190) (xy 58.2 198.08642)))
-    (crossbar (pts (xy 58.2 197.499999) (xy 97.2 197.499999)))
-    (arrow1a (pts (xy 97.2 197.499999) (xy 96.073496 198.08642)))
-    (arrow1b (pts (xy 97.2 197.499999) (xy 96.073496 196.913578)))
-    (arrow2a (pts (xy 58.2 197.499999) (xy 59.326504 198.08642)))
-    (arrow2b (pts (xy 58.2 197.499999) (xy 59.326504 196.913578)))
+    (feature1 (pts (xy 97.2 190) (xy 97.2 198.186421)))
+    (feature2 (pts (xy 58.2 190) (xy 58.2 198.186421)))
+    (crossbar (pts (xy 58.2 197.6) (xy 97.2 197.6)))
+    (arrow1a (pts (xy 97.2 197.6) (xy 96.073496 198.186421)))
+    (arrow1b (pts (xy 97.2 197.6) (xy 96.073496 197.013579)))
+    (arrow2a (pts (xy 58.2 197.6) (xy 59.326504 198.186421)))
+    (arrow2b (pts (xy 58.2 197.6) (xy 59.326504 197.013579)))
   )
   (dimension 19.5 (width 0.12) (layer Cmts.User)
@@
     (arrow2b (pts (xy 77.7 194.3) (xy 76.573496 194.886421)))
   )
-  (gr_line (start 311.7 191.5) (end 311.7 190) (layer Cmts.User) (width 0.12))
-  (gr_line (start 272.7 191.5) (end 272.7 190) (layer Cmts.User) (width 0.12))
-  (gr_line (start 233.7 191.5) (end 233.7 190) (layer Cmts.User) (width 0.12))
-  (gr_line (start 194.7 191.5) (end 194.7 190) (layer Cmts.User) (width 0.12))
-  (gr_line (start 155.7 191.5) (end 155.7 190) (layer Cmts.User) (width 0.12))
-  (gr_line (start 116.7 191.5) (end 116.7 190) (layer Cmts.User) (width 0.12))
   (gr_line (start 77.7 191.5) (end 77.7 190) (layer Cmts.User) (width 0.12))
-  (gr_line (start 331.2 191.5) (end 331.2 190) (layer Cmts.User) (width 0.12))
-  (gr_line (start 292.2 191.5) (end 292.2 190) (layer Cmts.User) (width 0.12))
-  (gr_line (start 253.2 191.5) (end 253.2 190) (layer Cmts.User) (width 0.12))
-  (gr_line (start 214.2 191.5) (end 214.2 190) (layer Cmts.User) (width 0.12))
-  (gr_line (start 175.2 191.5) (end 175.2 190) (layer Cmts.User) (width 0.12))
-  (gr_line (start 136.2 191.5) (end 136.2 190) (layer Cmts.User) (width 0.12))
   (gr_line (start 97.2 191.5) (end 97.2 190) (layer Cmts.User) (width 0.12))
   (gr_line (start 58.2 191.5) (end 58.2 190) (layer Cmts.User) (width 0.12))
-  (gr_line (start 58.2 191.5) (end 350.7 191.5) (layer Cmts.User) (width 0.12))
-  (gr_line (start 204.5 123.4) (end 204.5 204.2) (layer Cmts.User) (width 0.35))
   (gr_arc (start 362.98 77.270001) (end 364.250001 77.270001) (angle -90) (layer Edge.Cuts) (width 0.05))
   (gr_text "Interfacebox module board" (at 328.9 90.702) (layer F.SilkS)
@@
   (gr_line (start 44.6 184.53) (end 44.599999 77.270001) (layer Edge.Cuts) (width 0.05))
   (gr_circle (center 311.76 131.51) (end 307.71 135.42) (layer Edge.Cuts) (width 0.05))
-  (gr_text "35.5cm is box nu aan buitenkant (+4cm voor zijkant kabel uitsteeksel)\n    Hans: 1-2cm minder breed is fijn\n35.5 - 1 = 34.5 (door behuizing)\n34.5 - 2 = 32.5cm pcb?" (at 99.73 223.88) (layer Cmts.User)
+  (gr_text "35.5cm current box (+4cm on side for cable)\n    1-2cm less wide would fir better\n35.5 - 1 = 34.5 (housing = 1cm)\n34.5 - 2 = 32.5cm pcb" (at 99.73 223.88) (layer Cmts.User)
     (effects (font (size 1.5 1.5) (thickness 0.3)) (justify left))
   )
-  (gr_text "Preamp board ook modulair? \nHandig bij 'recycling' van box/preampboard\n\ngaten in pcb voor connectors\ngeen top ground waar module komt (tegen spikes)" (at 143.4 59.8) (layer Cmts.User)
-    (effects (font (size 1.5 1.5) (thickness 0.2)) (justify left))
-  )
   (gr_line (start 50.059 121.819) (end 93.62 121.819) (layer F.SilkS) (width 0.05))

Commit message: Added: holes for preamp socket pins, via's. Changed: 3D settings
Routing:
- net Net-(Ch16-Pad1): track 203.1 -> 205.2 mm
- net Net-(JP7-Pad2): track 139.1 -> 141.1 mm
- net Net-(JP5-Pad2): track 92.3 -> 94.4 mm
- net Net-(JP4-Pad2): track 70.7 -> 72.8 mm
- net Net-(Ch14-Pad1): track 176.0 -> 178.1 mm
- net Net-(Ch12-Pad1): track 180.7 -> 182.7 mm
- net Net-(Ch10-Pad1): track 158.6 -> 160.6 mm
- net Net-(JP3-Pad2): track 57.1 -> 59.1 mm
- net Net-(JP6-Pad2): track 116.0 -> 118.1 mm
- net Net-(Ch8-Pad1): track 222.9 -> 225.0 mm
- net GND: vias 131 -> 502
Other:
- board text added: "03/2020 v0.2"
- board text removed: "02/2020 v0.2"
