File: Interfacebox module board.kicad_pcb (KiCad board)
At the start: 2 copper layers, 319.7 x 109.8 mm, 88 parts, among them J1 Malfboard bottom, J2 Malfboard top, J3 Driverboard_malf-board, J4 Driverboard_TR-switch, J5 1-8, J6 9-16

Commit message: Added: mounting holes for 2 RXE4's
Parts:
- removed the H1 at (51.3, 78.6)
- removed H101 (x2), H102, H104, H105, H106, H107, H108, H3 (x2), H8: MH_Pad, _Custom:MountingHole_3.2mm_M3_plated
- removed the H2 at (51.3, 119.5)
- removed the H4 at (81.8, 78.6)
- added SYM3: RXE4, _Custom:RXE4, F.Cu at (287.8, 92.5)
- added SYM4: RXE4, _Custom:RXE4, F.Cu at (121.1, 92.5)
- added SYM5: RXE4, _Custom:RXE4, F.Cu at (122.6, 92.5)
- added SYM6: RXE4, _Custom:RXE4, F.Cu at (286.3, 92.5)
- moved H2 2.44 mm to (250.1, 81.0)
- moved Ch4 2.44 mm to (149.2, 99.0)
- moved J2 2.44 mm to (115.7, 80.7)
- moved Ch1 2.44 mm to (127.0, 99.0)
- moved Ch10 2.44 mm to (193.6, 99.0)
- moved Ch11 2.44 mm to (201.0, 99.0)
- moved Ch12 2.44 mm to (208.4, 99.0)
- moved Ch13 2.44 mm to (215.8, 99.0)
- moved Ch14 2.44 mm to (223.2, 99.0)
- moved Ch15 2.44 mm to (230.6, 99.0)
- moved Ch16 2.44 mm to (238.0, 99.0)
- moved Ch2 2.44 mm to (134.4, 99.0)
- moved Ch3 2.44 mm to (141.8, 99.0)
- moved Ch5 2.44 mm to (156.6, 99.0)
- moved Ch6 2.44 mm to (164.0, 99.0)
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Routing:
- net Net-(Ch10-Pad1): track 160.6 -> 166.7 mm
- net Net-(Ch16-Pad1): track 205.2 -> 210.0 mm
- net Net-(Ch14-Pad1): track 178.1 -> 182.5 mm
- net Net-(Ch9-Pad1): track 93.7 -> 97.4 mm
- net Net-(Ch6-Pad1): track 209.7 -> 213.2 mm
- net Net-(Ch7-Pad1): track 165.6 -> 168.9 mm
- net Net-(Ch12-Pad1): track 182.7 -> 186.0 mm
- net Net-(JP1-Pad2): track 75.6 -> 72.6 mm
- net Net-(Ch3-Pad1): track 163.7 -> 166.7 mm
- net Malf_MD: track 32.3 -> 29.8 mm
- net Ref_V+: track 17.7 -> 15.2 mm
- net Net-(JP5-Pad2): track 94.4 -> 96.8 mm
- net detune_in: track 41.2 -> 38.8 mm
- net Net-(JP7-Pad2): track 141.1 -> 143.6 mm
- net Net-(JP6-Pad2): track 118.1 -> 120.5 mm
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
Commit message: Changed: better and new footprint for malfunctionboard
Parts:
- removed Ch1, Ch10, Ch11, Ch12, Ch13, Ch14, Ch15, Ch16, Ch2, Ch3, Ch4, Ch5, Ch6, Ch7, Ch8, Ch9: Malf board, _Custom:Header_5.08mm_Drill1mm
- removed G1: LOGO, _Custom:UMC_logo
- removed J1: Malfboard bottom, Connector_IDC:IDC-Header_2x05_P2.54mm_Vertical
- removed J2: Malfboard top, Connector_IDC:IDC-Header_2x05_P2.54mm_Vertical
- removed J3: Driverboard_malf-board, Connector_IDC:IDC-Header_2x05_P2.54mm_Vertical
- removed SYM1: Driverboard, _Custom:Driverboard
- J4: footprint Connector_IDC:IDC-Header_2x07_P2.54mm_Vertical -> _Custom:Driverboard
- MB1: renamed from SYM2; value Malfunctionboard -> Malfboard
- moved J4 19.5 mm to (73.0, 100.5)
- moved MB1 0.09 mm to (173.0, 93.8)
Connections:
- J4 pad 1: Net-(J4-Pad1) -> Ref_V-
- J4 pad 10: Net-(J4-Pad10) -> GND
- J4 pad 11: Net-(J4-Pad11) -> GND
- J4 pad 12: Net-(J4-Pad12) -> GND
- J4 pad 2: Net-(J4-Pad2) -> Ref_V+
- J4 pad 3: GND -> Malf_MH
- J4 pad 4: GND -> Malf
- J4 pad 5: GND -> +12V
- J4 pad 6: GND -> -5V
- J4 pad 7: Net-(J4-Pad7) -> detune_in
- J4 pad 8: Net-(J4-Pad8) -> detune_in
- J4 pad 9: Net-(J4-Pad9) -> GND
- JP1 pad 1: Net-(Ch2-Pad1) -> Net-(JP1-Pad1)
- JP1 pad 3: Net-(Ch3-Pad1) -> Net-(JP1-Pad3)
- JP2 pad 1: Net-(Ch3-Pad1) -> Net-(JP1-Pad3)
- JP2 pad 3: Net-(Ch5-Pad1) -> Net-(JP2-Pad3)
- JP3 pad 1: Net-(Ch4-Pad1) -> Net-(JP3-Pad1)
- JP3 pad 3: Net-(Ch7-Pad1) -> Net-(JP3-Pad3)
- JP4 pad 1: Net-(Ch5-Pad1) -> Net-(JP2-Pad3)
- JP4 pad 3: Net-(Ch9-Pad1) -> Net-(JP4-Pad3)
- JP5 pad 1: Net-(Ch6-Pad1) -> Net-(JP5-Pad1)
- JP5 pad 3: Net-(Ch11-Pad1) -> Net-(JP5-Pad3)
- JP6 pad 1: Net-(Ch7-Pad1) -> Net-(JP3-Pad3)
- JP6 pad 3: Net-(Ch13-Pad1) -> Net-(JP6-Pad3)
- JP7 pad 1: Net-(Ch8-Pad1) -> Net-(JP7-Pad1)
- JP7 pad 3: Net-(Ch15-Pad1) -> Net-(JP7-Pad3)
- L1 pad 2: Net-(Ch1-Pad1) -> Net-(L1-Pad2)
- L10 pad 2: Net-(Ch10-Pad1) -> Net-(L10-Pad2)
- L11 pad 2: Net-(Ch11-Pad1) -> Net-(JP5-Pad3)
- L12 pad 2: Net-(Ch12-Pad1) -> Net-(L12-Pad2)
- L13 pad 2: Net-(Ch13-Pad1) -> Net-(JP6-Pad3)
- L14 pad 2: Net-(Ch14-Pad1) -> Net-(L14-Pad2)
- L15 pad 2: Net-(Ch15-Pad1) -> Net-(JP7-Pad3)
- L16 pad 2: Net-(Ch16-Pad1) -> Net-(L16-Pad2)
- L2 pad 2: Net-(Ch2-Pad1) -> Net-(JP1-Pad1)
- L3 pad 2: Net-(Ch3-Pad1) -> Net-(JP1-Pad3)
- L4 pad 2: Net-(Ch4-Pad1) -> Net-(JP3-Pad1)
- L5 pad 2: Net-(Ch5-Pad1) -> Net-(JP2-Pad3)
- L6 pad 2: Net-(Ch6-Pad1) -> Net-(JP5-Pad1)
- L7 pad 2: Net-(Ch7-Pad1) -> Net-(JP3-Pad3)
- L8 pad 2: Net-(Ch8-Pad1) -> Net-(JP7-Pad1)
- L9 pad 2: Net-(Ch9-Pad1) -> Net-(JP4-Pad3)
- MB1 pad 1: (no net) -> GND
- Preampboard-1 pad 2: Net-(Ch1-Pad1) -> Net-(L1-Pad2)
- Preampboard-10 pad 2: Net-(Ch10-Pad1) -> Net-(L10-Pad2)
- Preampboard-12 pad 2: Net-(Ch12-Pad1) -> Net-(L12-Pad2)
- Preampboard-14 pad 2: Net-(Ch14-Pad1) -> Net-(L14-Pad2)
- Preampboard-16 pad 2: Net-(Ch16-Pad1) -> Net-(L16-Pad2)
- Preampboard-2 pad 2: Net-(Ch2-Pad1) -> Net-(JP1-Pad1)
- Preampboard-4 pad 2: Net-(Ch4-Pad1) -> Net-(JP3-Pad1)
- Preampboard-6 pad 2: Net-(Ch6-Pad1) -> Net-(JP5-Pad1)
- Preampboard-8 pad 2: Net-(Ch8-Pad1) -> Net-(JP7-Pad1)
Routing:
- net Net-(L1-Pad2): track 0.00 -> 256.8 mm
- net Net-(Ch1-Pad1): track 256.8 -> 0.00 mm
- net Net-(JP1-Pad1): track 0.00 -> 247.3 mm
- net Net-(Ch2-Pad1): track 247.3 -> 0.00 mm
- net Net-(JP3-Pad1): track 0.00 -> 235.9 mm, vias 0 -> 3
- net Net-(Ch4-Pad1): track 235.9 -> 0.00 mm, vias 3 -> 0
- net Net-(JP7-Pad1): track 0.00 -> 227.4 mm, vias 0 -> 3
- net Net-(Ch8-Pad1): track 227.4 -> 0.00 mm, vias 3 -> 0
- net Net-(JP5-Pad1): track 0.00 -> 213.2 mm, vias 0 -> 1
- net Net-(Ch6-Pad1): track 213.2 -> 0.00 mm, vias 1 -> 0
- net Net-(L16-Pad2): track 0.00 -> 210.0 mm
- net Net-(Ch16-Pad1): track 210.0 -> 0.00 mm
- net Net-(L12-Pad2): track 0.00 -> 186.0 mm, vias 0 -> 2
- net Net-(Ch12-Pad1): track 186.0 -> 0.00 mm, vias 2 -> 0
- net Net-(L14-Pad2): track 0.00 -> 182.5 mm
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Other:
- rule via_min_drill: 0.3 -> 0.25

Commit message: Updated: preamp footprint to accommodate preci-dip connectors. Added: some GND via's
Routing:
- net Net-(JP5-Pad1): track 213.2 -> 212.3 mm
- net Net-(JP3-Pad1): track 235.9 -> 235.0 mm
- net GND: vias 516 -> 517

Commit message: Added: missing logo
Parts:
- added G1: UMC_logo, _Custom:UMC_logo_small, F.Cu at (325.8, 92.7)

Commit message: Small changes. V0.3
Parts:
- J4: value Driverboard_TR-switch -> Driverboard
Routing:
- net GND: vias 517 -> 0
- net (no net): vias 0 -> 1
- removed copper zone on F.Cu, net GND
Other:
- board text added: "04/2020 v0.3"
- board text added: "Connect J6 on master to J5 on slave board to make 2x8ch"
- board text removed: "03/2020 v0.2"
- board text removed: "Connect J6 on master to J5 on slave board to make 16ch with 1 driver/malfunction board"

Commit message: v0.3
Other:
- rule pad_to_mask_clearance: 0.051 -> 0

Commit message: Updated to v1.0
Other:
- board text added: "11/2021 v1.0"
- board text removed: "04/2020 v0.3"
